File: projetos/descongestionator/kicad_project/kicad_project.kicad_sch (KiCad schematic)
At the start: 21 parts, among them J1 USB_A, J2 Conn_01x05_Socket, Q1 PN2222A, U1 LCD-016N002L, U2 PCF8574, U3 CP2102N-Axx-xQFN20

Commit message: gps e MCU
Parts:
- added J3: U.FL-R-SMT_01_, components_kicad:HRS_U.FL-R-SMT_01_, symbol U.FL-R-SMT_01_:U.FL-R-SMT_01_
- added R10, R11, R9: 10k, symbol Device:R
- added U4: NEO-6M-GPS, components_kicad:XCVR_NEO-6M-GPS, symbol NEO-6M-GPS:NEO-6M-GPS
- added U5: ATtiny202-SS, Package_SO:SOIC-8_3.9x4.9mm_P1.27mm, symbol MCU_Microchip_ATtiny:ATtiny202-SS
Connections:
- net +3V3: now also R10.1, R11.1, R9.1, U4.23 (VCC), U5.1 (VCC)
- net GND: now also J3.1 (GND), J3.2 (GND), U4.10 (GND), U4.12 (GND), U4.13 (GND), U4.24 (GND), U5.8 (GND)
- net at U2.14 (SCL): now also J2.3 (Pin_3), R11.2, U4.19 (SCL2), U5.5 (PA2)
- net at U2.15 (SDA): now also J2.4 (Pin_4), R10.2, U4.18 (SDA2), U5.4 (PA1)
- net at R8.2: now also U5.7 (PA3)
- net at U3.17 (RXD): now also U5.2 (PA6)
- net at U3.18 (TXD): now also U5.3 (PA7)
- new net: J3.3 (SIG), U4.11 (RF_IN)
- new net: U4.8 (RSVD_8), U4.9 (VCC_RF)
- new net: R9.2, U5.6 (~{RESET}/PA0)
Other:
- note added: "MCU"
- note added: "RX"
- note added: "TX"
- note added: "chip GPS + Antena"
- moved on the sheet: BZ1, C1, C2, C3, C4, D1, J1, J2, Q1, R5, R6, R7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

Commit message: roteamento + modelos 3d
Parts:
- BZ1: footprint (none) -> Buzzer_Beeper:Buzzer_12x9.5RM7.6
- C1, C2, C3, C4: footprint (none) -> Capacitor_SMD:C_0402_1005Metric_Pad0.74x0.62mm_HandSolder
- J1: footprint (none) -> Connector_USB:USB_A_Receptacle_GCT_USB1046
- J2: footprint (none) -> Connector_TE-Connectivity:TE_826576-5_1x05_P3.96mm_Vertical
- R1, R10, R11, R2, R3, R5, R6, R7, R8, R9: footprint (none) -> Resistor_SMD:R_0402_1005Metric
- R4: footprint (none) -> Resistor_SMD:R_0603_1608Metric_Pad0.98x0.95mm_HandSolder
- RV1: footprint (none) -> Potentiometer_SMD:Potentiometer_Bourns_3214G_Horizontal
- U2: footprint (none) -> Package_DFN_QFN:VQFN-16-1EP_3x3mm_P0.5mm_EP1.8x1.8mm
- U3: footprint Package_DFN_QFN:SiliconLabs_QFN-20-1EP_3x3mm_P0.5mm -> Package_DFN_QFN:QFN-20-1EP_3x3mm_P0.45mm_EP1.6x1.6mm
Other:
- moved on the sheet: J3
Changed lines of the file:
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@@
 	(wire
 		(pts
-			(xy 246.38 96.52) (xy 254 96.52)
+			(xy 246.38 96.52) (xy 251.46 96.52)
 		)
 		(stroke
@@
 			)
 		)
-		(property "Footprint" ""
+		(property "Footprint" "Resistor_SMD:R_0402_1005Metric"
 			(at 182.118 39.37 90)
 			(effects
@@
 			)
 		)
-		(property "Footprint" ""
+		(property "Footprint" "Resistor_SMD:R_0402_1005Metric"
 			(at 173.228 39.37 90)
 			(effects
@@
 			)
 		)
-		(property "Footprint" ""
+		(property "Footprint" "Package_DFN_QFN:VQFN-16-1EP_3x3mm_P0.5mm_EP1.8x1.8mm"
 			(at 205.74 45.72 0)
 			(effects
@@
 			)
 		)
-		(property "Footprint" ""
+		(property "Footprint" "Resistor_SMD:R_0402_1005Metric"
 			(at 49.022 58.42 90)
 			(effects
@@
 			)
 		)
-		(property "Footprint" ""
+		(property "Footprint" "Potentiometer_SMD:Potentiometer_Bourns_3214G_Horizontal"
 			(at 265.43 30.48 0)
 			(effects
@@
 			)
 		)
-		(property "Footprint" ""
+		(property "Footprint" "Capacitor_SMD:C_0402_1005Metric_Pad0.74x0.62mm_HandSolder"
 			(at 61.9252 36.83 0)
 			(effects
@@
 			)
 		)
-		(property "Footprint" ""
+		(property "Footprint" "Resistor_SMD:R_0402_1005Metric"
 			(at 169.672 76.2 90)
 			(effects
@@
 			)
 		)
-		(property "Footprint" ""
+		(property "Footprint" "Capacitor_SMD:C_0402_1005Metric_Pad0.74x0.62mm_HandSolder"
 			(at 77.1652 36.83 0)
 			(effects
@@
 			)
 		)
-		(property "Footprint" ""
+		(property "Footprint" "Resistor_SMD:R_0402_1005Metric"
 			(at 49.022 66.04 90)
 			(effects
@@
 			)
 		)
-		(property "Footprint" ""
+		(property "Footprint" "Connector_TE-Connectivity:TE_826576-5_1x05_P3.96mm_Vertical"
 			(at 213.36 153.67 0)
 			(effects
@@
 			)
 		)
-		(property "Footprint" ""
+		(property "Footprint" "Resistor_SMD:R_0402_1005Metric"
 			(at 133.858 148.59 90)
 			(effects
@@
 			)
 		)
-		(property "Footprint" "Package_DFN_QFN:SiliconLabs_QFN-20-1EP_3x3mm_P0.5mm"
+		(property "Footprint" "Package_DFN_QFN:QFN-20-1EP_3x3mm_P0.45mm_EP1.6x1.6mm"
 			(at 104.14 106.68 0)
 			(effects
@@
 			)
 		)
-		(property "Footprint" ""
+		(property "Footprint" "Capacitor_SMD:C_0402_1005Metric_Pad0.74x0.62mm_HandSolder"
 			(at 88.5952 36.83 0)
 			(effects
@@
 			)
 		)
-		(property "Footprint" ""
+		(property "Footprint" "Capacitor_SMD:C_0402_1005Metric_Pad0.74x0.62mm_HandSolder"
 			(at 51.7652 36.83 0)
 			(effects
@@
 			)
 		)
-		(property "Footprint" ""
+		(property "Footprint" "Resistor_SMD:R_0402_1005Metric"
 			(at 56.642 49.53 90)
 			(effects
@@
 			)
 		)
-		(property "Footprint" ""
+		(property "Footprint" "Resistor_SMD:R_0402_1005Metric"
 			(at 178.562 76.2 90)
 			(effects
@@
 			)
 		)
-		(property "Footprint" ""
+		(property "Footprint" "Resistor_SMD:R_0603_1608Metric_Pad0.98x0.95mm_HandSolder"
 			(at 277.368 30.48 90)
 			(effects
@@
 	(symbol
 		(lib_id "power:GND")
-		(at 254 101.6 0)
+		(at 251.46 101.6 0)
 		(unit 1)
 		(exclude_from_sim no)
@@
 		(fields_autoplaced yes)
 		(property "Reference" "#PWR017"
-			(at 254 107.95 0)
+			(at 251.46 107.95 0)
 			(effects
 				(font
@@
 		)
 		(property "Value" "GND"
-			(at 254 106.68 0)
+			(at 251.46 106.68 0)
 			(effects
 				(font
@@
 		)
 		(property "Footprint" ""
-			(at 254 101.6 0)
+			(at 251.46 101.6 0)
 			(effects
 				(font
@@
 		)
 		(property "Datasheet" ""
-			(at 254 101.6 0)
+			(at 251.46 101.6 0)
 			(effects
 				(font
@@
 		)
 		(property "Description" "Power symbol creates a global label with name \"GND\" , ground"
-			(at 254 101.6 0)
+			(at 251.46 101.6 0)
 			(effects
 				(font
@@
 			)
 		)
-		(property "Footprint" ""
+		(property "Footprint" "Resistor_SMD:R_0402_1005Metric"
 			(at 154.432 76.2 90)
 			(effects
@@
 	(symbol
 		(lib_id "U.FL-R-SMT_01_:U.FL-R-SMT_01_")
-		(at 264.16 99.06 0)
+		(at 261.62 99.06 0)
 		(unit 1)
 		(exclude_from_sim no)
@@
 		(fields_autoplaced yes)
 		(property "Reference" "J3"
-			(at 270.51 98.0439 0)
+			(at 267.97 98.0439 0)
 			(effects
 				(font
@@
 		)
 		(property "Value" "U.FL-R-SMT_01_"
-			(at 270.51 100.5839 0)
+			(at 267.97 100.5839 0)
 			(effects
 				(font
@@
 		)
 		(property "Footprint" "components_kicad:HRS_U.FL-R-SMT_01_"
-			(at 264.16 99.06 0)
+			(at 261.62 99.06 0)
 			(effects
 				(font
@@
 		)
 		(property "Datasheet" ""
-			(at 264.16 99.06 0)
+			(at 261.62 99.06 0)
 			(effects
 				(font
@@
 		)
 		(property "Description" ""
-			(at 264.16 99.06 0)
+			(at 261.62 99.06 0)
 			(effects
 				(font
@@
 		)
 		(property "MF" "Hirose"
-			(at 264.16 99.06 0)
+			(at 261.62 99.06 0)
 			(effects
 				(font
@@
 		)
 		(property "DESCRIPTION" "U.FL Series 6 Ghz 50 Ohm Ultra-small SMT Coaxial Cable Receptacle"
-			(at 264.16 99.06 0)
+			(at 261.62 99.06 0)
 			(effects
 				(font
@@
 		)
 		(property "PACKAGE" "None"
-			(at 264.16 99.06 0)
+			(at 261.62 99.06 0)
 			(effects
 				(font
@@
 		)
 		(property "PRICE" "0.84 USD"
-			(at 264.16 99.06 0)
+			(at 261.62 99.06 0)
 			(effects
 				(font
@@
 		)
 		(property "Package" "None"
-			(at 264.16 99.06 0)
+			(at 261.62 99.06 0)
 			(effects
 				(font
@@
 		)
 		(property "Check_prices" "https://www.snapeda.com/parts/U.FL-R-SMT(01)/Hirose+Electric+Co+Ltd/view-part/?ref=eda"
-			(at 264.16 99.06 0)
+			(at 261.62 99.06 0)
 			(effects
 				(font
@@
 		)
 		(property "Price" "None"
-			(at 264.16 99.06 0)
+			(at 261.62 99.06 0)
 			(effects
 				(font
@@
 		)
 		(property "SnapEDA_Link" "https://www.snapeda.com/parts/U.FL-R-SMT(01)/Hirose+Electric+Co+Ltd/view-part/?ref=snap"
-			(at 264.16 99.06 0)
+			(at 261.62 99.06 0)
 			(effects
 				(font
@@
 		)
 		(property "MP" "U.FL-R-SMT(01)"
-			(at 264.16 99.06 0)
+			(at 261.62 99.06 0)
 			(effects
 				(font
@@
 		)
 		(property "Purchase-URL" "https://www.snapeda.com/api/url_track_click_mouser/?unipart_id=49572&manufacturer=Hirose&part_name=U.FL-R-SMT(01)&search_term=None"
-			(at 264.16 99.06 0)
+			(at 261.62 99.06 0)
 			(effects
 				(font
@@
 		)
 		(property "Availability" "In Stock"
-			(at 264.16 99.06 0)
+			(at 261.62 99.06 0)
 			(effects
 				(font
@@
 		)
 		(property "AVAILABILITY" "Good"
-			(at 264.16 99.06 0)
+			(at 261.62 99.06 0)
 			(effects
 				(font
@@
 		)
 		(property "Description_1" "\nU.FL (UMCC) Connector Receptacle, Male Pin 50Ohm Surface Mount Solder. RF Connectors / Coaxial Connectors\n"
-			(at 264.16 99.06 0)
+			(at 261.62 99.06 0)
 			(effects
 				(font
@@
 			)
 		)
-		(property "Footprint" ""
+		(property "Footprint" "Connector_USB:USB_A_Receptacle_GCT_USB1046"
 			(at 34.29 76.2 0)
 			(effects
@@
 			)
 		)
-		(property "Footprint" ""
+		(property "Footprint" "Resistor_SMD:R_0402_1005Metric"
 			(at 164.338 39.37 90)
 			(effects
@@
 			)
 		)
-		(property "Footprint" ""
+		(property "Footprint" "Buzzer_Beeper:Buzzer_12x9.5RM7.6"
 			(at 144.145 143.51 90)
 			(effects

Commit message: esquema eletrico pdf
Other:
- company: (none) -> EA075 UNICAMP CaseTars
- title: (none) -> Projeto Descongestionator
Changed lines of the file:
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@@
 	(generator_version "8.0")
 	(paper "A4")
+	(title_block
+		(title "Projeto Descongestionator")
+		(date "2024-06-24")
+		(company "EA075 UNICAMP CaseTars")
+	)
 	(junction
 		(at 60.96 36.83)
